Commit message: Fix differential turning and validate optional sensors and RViz

File: src/limo_autorace_sim/urdf/limo_sim.xacro (robot description, xacro)
@@ -40,5 +40,7 @@
       <limit effort="${v['wheel_effort']}" velocity="50"/><dynamics damping="0.001" friction="0"/>
     </joint>
-    <gazebo reference="${name}_wheel_link"><mu1>${v['wheel_friction']}</mu1><mu2>${v['wheel_friction']}</mu2><kp>100000</kp><kd>10</kd><minDepth>0.0001</minDepth><maxVel>0.1</maxVel></gazebo>
+    <!-- Collision-local Z is parallel to the wheel axle after its pi/2 rotation.
+         WheelSlip requires fdir1 along that axle: slip1=lateral, slip2=rolling. -->
+    <gazebo reference="${name}_wheel_link"><mu1>${v['wheel_friction']}</mu1><mu2>${v['wheel_friction']}</mu2><fdir1>0 0 1</fdir1><kp>100000</kp><kd>10</kd><minDepth>0.0001</minDepth><maxVel>0.1</maxVel></gazebo>
   </xacro:macro>
   <xacro:wheel name="rear_left" x="0" side="${1}" front="${False}"/>
@@ -71,5 +73,5 @@
   <gazebo>
     <plugin filename="gz-sim-wheel-slip-system" name="gz::sim::systems::WheelSlip">
-      <xacro:macro name="slip_wheel" params="name"><wheel link_name="${name}_wheel_link"><slip_compliance_lateral>${v['wheel_slip']}</slip_compliance_lateral><slip_compliance_longitudinal>${v['wheel_slip']}</slip_compliance_longitudinal><wheel_normal_force>${(v['body_mass']+4*v['wheel_mass']+2*v['hinge_mass'])*9.80665/4}</wheel_normal_force><wheel_radius>${R}</wheel_radius></wheel></xacro:macro>
+      <xacro:macro name="slip_wheel" params="name"><wheel link_name="${name}_wheel_link"><slip_compliance_lateral>${v['wheel_slip'] if ack else v.get('diff_lateral_slip', 1.0)}</slip_compliance_lateral><slip_compliance_longitudinal>${v['wheel_slip']}</slip_compliance_longitudinal><wheel_normal_force>${(v['body_mass']+4*v['wheel_mass']+(2*v['hinge_mass'] if ack else 0))*9.80665/4}</wheel_normal_force><wheel_radius>${R}</wheel_radius></wheel></xacro:macro>
       <xacro:slip_wheel name="front_left"/><xacro:slip_wheel name="front_right"/><xacro:slip_wheel name="rear_left"/><xacro:slip_wheel name="rear_right"/>
     </plugin>
